File: schematic/receiver.sch (EAGLE design)
At the start: 4 parts

Commit message: updated schematic: added attiny85
Parts:
- added U$2: ATTINY85, stuff:ATTINY85
Connections:
- net ARDUINO_PIN_0: now also U$2.PIN0
- net ARDUINO_PIN_1: now also U$2.PIN1
- net ARDUINO_PIN_GND: now also U$2.GND
- net ARDUINO_PIN_VIN: now also U$2.VCC
Changed lines of the file:
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@@
 <part name="SUPPLY1" library="supply2" deviceset="+7V" device=""/>
 <part name="GND3" library="supply1" deviceset="GND" device=""/>
+<part name="U$2" library="stuff" deviceset="ATTINY85" device=""/>
 </parts>
 <sheets>
@@
 <instance part="SUPPLY1" gate="G$1" x="-58.42" y="33.02"/>
 <instance part="GND3" gate="1" x="-58.42" y="0"/>
+<instance part="U$2" gate="G$1" x="38.1" y="43.18"/>
 </instances>
 <busses>
@@
 <pinref part="U$1" gate="G$1" pin="DIGITAL_OUT"/>
 <wire x1="-17.78" y1="25.4" x2="-17.78" y2="12.7" width="0.1524" layer="91"/>
-<wire x1="-17.78" y1="12.7" x2="25.4" y2="12.7" width="0.1524" layer="91"/>
-<label x="27.94" y="12.7" size="1.778" layer="95"/>
+<wire x1="-17.78" y1="12.7" x2="53.34" y2="12.7" width="0.1524" layer="91"/>
+<pinref part="U$2" gate="G$1" pin="PIN0"/>
+<wire x1="53.34" y1="12.7" x2="53.34" y2="33.02" width="0.1524" layer="91"/>
 </segment>
 </net>
@@
 <wire x1="-35.56" y1="2.54" x2="-35.56" y2="5.08" width="0.1524" layer="91"/>
 <junction x="-35.56" y="5.08"/>
-<wire x1="-20.32" y1="5.08" x2="25.4" y2="5.08" width="0.1524" layer="91"/>
-<label x="27.94" y="5.08" size="1.778" layer="95"/>
+<wire x1="-20.32" y1="5.08" x2="22.86" y2="5.08" width="0.1524" layer="91"/>
 <junction x="-20.32" y="5.08"/>
+<pinref part="U$2" gate="G$1" pin="GND"/>
+<wire x1="22.86" y1="5.08" x2="22.86" y2="33.02" width="0.1524" layer="91"/>
 </segment>
 </net>
@@
 <segment>
 <pinref part="R1" gate="G$1" pin="2"/>
-<wire x1="-12.7" y1="-5.08" x2="25.4" y2="-5.08" width="0.1524" layer="91"/>
-<label x="27.94" y="-5.08" size="1.778" layer="95"/>
+<wire x1="-12.7" y1="-5.08" x2="55.88" y2="-5.08" width="0.1524" layer="91"/>
+<wire x1="55.88" y1="-5.08" x2="55.88" y2="38.1" width="0.1524" layer="91"/>
+<pinref part="U$2" gate="G$1" pin="PIN1"/>
+<wire x1="55.88" y1="38.1" x2="53.34" y2="38.1" width="0.1524" layer="91"/>
 </segment>
 </net>
@@
 <wire x1="-12.7" y1="20.32" x2="-35.56" y2="20.32" width="0.1524" layer="91"/>
 <pinref part="VOLTAGE_REGULATOR" gate="A1" pin="VO"/>
-<wire x1="-12.7" y1="20.32" x2="25.4" y2="20.32" width="0.1524" layer="91"/>
-<label x="27.94" y="20.32" size="1.778" layer="95"/>
+<wire x1="-12.7" y1="20.32" x2="58.42" y2="20.32" width="0.1524" layer="91"/>
+<wire x1="58.42" y1="20.32" x2="58.42" y2="48.26" width="0.1524" layer="91"/>
+<pinref part="U$2" gate="G$1" pin="VCC"/>
+<wire x1="58.42" y1="48.26" x2="53.34" y2="48.26" width="0.1524" layer="91"/>
 </segment>
 </net>
